File: Zender/m06-zender/m06-zender.kicad_sch (KiCad schematic)
At the start: 17 parts, among them Q1 NPN, U1 TLV2371D

Commit message: 2nd version
Parts:
- removed L1: 15.9u, symbol Device:L
- removed Q1: NPN, symbol Simulation_SPICE:NPN
- removed U1: TLV2371D, Package_SO:SOIC-8_3.9x4.9mm_P1.27mm, symbol Amplifier_Operational:TLV2371D
- added C6, C7: 100n, symbol Device:C
- added D1, D2: 1N4148, Diode_THT:D_DO-35_SOD27_P7.62mm_Horizontal, symbol Diode:1N4148
- added R10, R11, R12, R14, R15, R16: 10k, symbol Device:R
- added R13: 38k, symbol Device:R
- added R17, R18, R19: 1k, symbol Device:R
- added RV1: 25k, symbol Device:R_Potentiometer
- added SW1, SW2: SW_Push, symbol Switch:SW_Push
- added U1: 40106, symbol 4xxx:40106
- added U2: 4066, symbol 4xxx:4066
- added U3: TL072, symbol Amplifier_Operational:TL072
- added U4: 4081, symbol 4xxx:4081
- C1: value 100n -> 100p
- C3, C5: value 470p -> 100n
- C4: value 1.59n -> 100n
- R2: value 40k -> 10k
- R3: value R -> 2k
- R4: value 4.7k -> 10k
- R5: value 1k -> 560
- R6: value 10k -> 2k
- R7: value 20k -> 10k
- R8: value 1k -> 22k
- R9: value 1k -> 10k
Connections:
- net AM Signal is gone; now on net GND: C5.2
- net +9V: now also C4.1, C5.1, R9.1, C6.1, C7.1, R11.1, R15.1, U1.14 (VDD), U2.14 (VDD), U3.8 (V+), U4.14 (VDD); no longer R7.1
- net GND: now also C6.2, C7.2, R10.2, R12.2, R14.2, R16.2, SW1.1, SW2.1, U1.7 (VSS), U2.7 (VSS), U3.4 (V-), U4.7 (VSS); no longer R3.2, R6.2, R9.2
- net at R4.1: now also U2.4; no longer C1.1
- net at R8.1: now also R7.1, U3.6 (-); no longer R9.1
- net at R8.2: now also R11.2, R12.1; no longer C5.1
- net at C3.1: now also R7.2, U3.7; no longer R1.2
- net Carrier signal renamed Carrier_Wave
- net Carrier_Wave: now also R13.2, R14.1
- net Data signal: no longer names the net of R4.2
- net Data signal: now also R3.2, R5.2, R9.2, R10.1
- new net: R6.2, U3.1, U3.5 (+)
- new net: R17.2, U2.6
- new net: R5.1, U2.8
- new net: D1.1 (K), D2.1 (K), U1.5
- new net: C2.2, R15.2, R16.1, U3.3 (+)
- new net: R18.2, U2.5
- new net: R19.2, U2.13
- new net: R2.2, SW2.2, U1.11
- new net: C1.1, RV1.3, U1.1
- new net: RV1.1, RV1.2, U1.2, U1.3
- new net: R3.1, U2.2
- new net: R13.1, U1.4
- new net BTN1: D1.2 (A), R18.1, U1.8
- new net BTN1_INV: R1.2, SW1.2, U1.9, U4.1
- new net BTN2: U1.10, U4.2
- new net BTN2_SOLO: D2.2 (A), R17.1, U4.3
- new net NO_BTN: R19.1, U1.6
- new net Resistor_Selector: R6.1, U2.1, U2.3, U2.9, U3.2 (-)
- new net SIGNAL_OUT: C3.2

Commit message: Final design modulator
Parts:
- removed R14: 10k, symbol Device:R
- added C8, C9: 100n, symbol Device:C
- added D3, D4: 1N4148, Diode_THT:D_DO-35_SOD27_P7.62mm_Horizontal, symbol Diode:1N4148
- added U5: 4020, symbol 4xxx:4020
- R10, R9: value 10k -> 1k
- R13: value 38k -> 10k
- R3: value 2k -> 10k
- R5: value 560 -> 10k
Connections:
- net +9V: now also U5.16 (VDD); no longer R9.1
- net BTN1_INV: now also R9.2, C8.2; no longer R1.2, SW1.2
- net Carrier_Wave: now also D3.2 (A)
- net GND: now also C8.1, C9.1, D4.1 (K), U5.11 (Reset), U5.8 (VSS); no longer R10.2
- net at U2.4: now also R4.2; no longer R4.1
- net SIGN-WAVE-SELECTED: now reaches R5.1
- net SIGN-WAVE-SELECTED: now also R3.1, R4.1, R6.1, U3.2 (-); no longer U2.8
- net at R2.2, SW2.2: now also R10.1; no longer U1.11
- net at U2.2: now also R3.2; no longer R3.1
- net 1MHz-Block: now reaches R13.1, U1.4
- net 1MHz-Block: now also U5.10 (CLK)
- removed net Resistor_Selector: R6.1, U2.1, U2.3, U2.9, U3.2 (-)
- new net: R5.2, U2.9
- new net: C9.2, R10.2, U1.11
- new net: D3.1 (K), D4.2 (A)
- new net: R1.2, R9.1, SW1.2
- new net SIGN-WAVE-FAST: U2.3, U5.7 (Q3)
- new net SIGN-WAVE-MED: U2.1, U5.5 (Q4)
- new net SIGN-WAVE-SLOW: U2.8, U5.4 (Q5)
Other:
- moved on the sheet: C1, C2, C3, C4, C5, C6, C7, D1, D2, R11, R12, R13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
